Commit message: adding

File: install/my_rover/share/my_rover/urdf/cam.xacro (robot description, xacro)
@@ -26,5 +26,5 @@
                 <clip>
                     <near>0.02</near>
-                    <far>300</far>
+                    <far>1000</far>
                 </clip>
                 <noise>
@@ -37,5 +37,5 @@
                 <frame_name>camera_link</frame_name>
                 <min_depth>0.1</min_depth>
-                <max_depth>500</max_depth>
+                <max_depth>1000</max_depth>
             </plugin>
         </sensor>

File: install/my_rover/share/my_rover/urdf/gps.xacro (robot description, xacro)
@@ -24,8 +24,8 @@
     </xacro:inertial_cylinder>
   </link>
-<gazebo reference="gps_link">
+  <gazebo reference="gps_link">
     <sensor name="gps_sensor" type="gps">
         <always_on>true</always_on>
-        <update_rate>1.0</update_rate>
+        <update_rate>10.0</update_rate>
         <plugin name="gps_controller" filename="libgazebo_ros_gps_sensor.so">
             <ros>
@@ -34,7 +34,9 @@
             </ros>
             <frame_name>gps_link</frame_name>
+            <horizontal_position_std_dev>0.0</horizontal_position_std_dev>
+            <vertical_position_std_dev>0.0</vertical_position_std_dev>
         </plugin>
     </sensor>
     <material>Gazebo/Grey</material>
-</gazebo>
+  </gazebo>
   </robot>

File: install/my_rover/share/my_rover/urdf/lidar.xacro (robot description, xacro)
@@ -30,36 +30,36 @@
   <gazebo reference="laser_frame">
     <sensor name="lidar" type="ray">
-    <pose>0.215 0 0.215 0 0 0</pose>
-    <always_on>true</always_on>
-    <visualize>true</visualize>
-    <update_rate>5</update_rate>
-    <ray>
-      <scan>
-        <horizontal>
-          <samples>360</samples>
-          <resolution>1.00000</resolution>
-          <min_angle>0.000000</min_angle>
-          <max_angle>6.280000</max_angle>
-        </horizontal>
-      </scan>
-      <range>
-        <min>0.120000</min>
-        <max>3.5</max>
-        <resolution>0.015000</resolution>
-      </range>
-      <noise>
-        <type>gaussian</type>
-        <mean>0.0</mean>
-        <stddev>0.01</stddev>
-      </noise>
-    </ray>
-    <plugin name="scan" filename="libgazebo_ros_ray_sensor.so">
-      <ros>
-        <remapping>~/out:=scan</remapping>
-      </ros>
-      <output_type>sensor_msgs/LaserScan</output_type>
-      <frame_name>laser_frame</frame_name>
-    </plugin>
-  </sensor>
+      <pose>0.215 0 0.215 0 0 0</pose>
+      <always_on>true</always_on>
+      <visualize>true</visualize>
+      <update_rate>5</update_rate>
+      <ray>
+        <scan>
+          <horizontal>
+            <samples>360</samples>
+            <resolution>1.00000</resolution>
+            <min_angle>0.000000</min_angle>
+            <max_angle>6.280000</max_angle>
+          </horizontal>
+        </scan>
+        <range>
+          <min>0.120000</min>
+          <max>3.5</max>
+          <resolution>0.015000</resolution>
+        </range>
+        <noise>
+          <type>gaussian</type>
+          <mean>0.0</mean>
+          <stddev>0.01</stddev>
+        </noise>
+      </ray>
+      <plugin name="scan" filename="libgazebo_ros_ray_sensor.so">
+        <ros>
+          <remapping>~/out:=scan</remapping>
+        </ros>
+        <output_type>sensor_msgs/LaserScan</output_type>
+        <frame_name>laser_frame</frame_name>
+      </plugin>
+    </sensor>
   </gazebo>
 </robot>

File: install/my_rover/share/my_rover/urdf/robot.urdf.xacro (robot description, xacro)
@@ -27,5 +27,4 @@
         <color rgba = "0.7 0.9 0 1" />
     </material>
-    <!-- Define base_footprint -->
     <link name="base_footprint">
         <inertial>
@@ -35,4 +34,9 @@
         </inertial>
     </link>
+    <joint name="base_joint" type="fixed">
+        <parent link="base_footprint"/>
+        <child link="base_link"/>
+        <origin xyz = "0 0 0.05" rpy = "0 0 0" />
+    </joint>
     <link name = "base_link">
         <visual>
@@ -53,10 +57,4 @@
         </xacro:inertial_box>
     </link>
-    <!-- Fixed joint to attach base_footprint to base_link -->
-    <joint name="base_link_to_base_footprint" type="fixed">
-        <parent link="base_footprint"/>
-        <child link="base_link"/>
-        <origin xyz="0 0 0.05" rpy="0 0 0"/>
-    </joint>
     <gazebo reference="base_link">
         <material>Gazebo/Red</material>
@@ -198,5 +196,5 @@
         </plugin>
     </gazebo>
-        <gazebo>
+    <gazebo>
         <plugin name="gazebo_ros_joint_state_publisher" filename="libgazebo_ros_joint_state_publisher.so">
             <update_rate>10</update_rate>
